Commit message: Messhes added into mobile_base pkg

File: catkin_ws/src/mobile_base/urdf/R2D2.urdf (robot description, URDF)
Before this commit: robot R2D2, 16 links, 15 joints
Links:
- added link laser_link
Joints:
- added joint laser_joint: type fixed, parent base_link, child laser_link, origin xyz=0.06323 0 0.04 rpy=0 0 0, axis 0 0 0

File: catkin_ws/src/mobile_base/urdf/six_w.urdf (robot description, URDF)
Before this commit: robot six_w, 7 links, 6 joints
Links:
- added link laser_link
Joints:
- added joint laser_joint: type fixed, parent base_link, child laser_link, origin xyz=0.06323 0 0.04 rpy=0 0 0, axis 0 0 0
