Commit message: Added real mesh into rviz visualization

File: catkin_ws/src/mobile_base/urdf/carritoAP.urdf (robot description, URDF)
Before this commit: robot carritoAP, 6 links, 5 joints
Links:
- link base_link: geometry visual mesh filename=package://mobile_base/stl/carritoAP.stl
- link free_frontal_wheel_link: geometry 
- link free_rear_wheel_link: geometry 
- link left_wheel_link: geometry 
- link right_wheel_link: geometry 
